Commit message: sample complete URDF and a readme with explanation

File: src/URDF/my_robot.urdf (robot description, URDF)
Before this commit: robot my_robot, 2 links, 1 joints
Links:
- added link base_footprint
- added link caster_wheel; visual sphere radius=0.05
- added link left_wheel; visual cylinder length=0.05 radius=0.1
- added link right_wheel; visual cylinder length=0.05 radius=0.1
Joints:
- removed joint laser_joint
- added joint base_caster_wheel_joint: type fixed, parent base_link, child caster_wheel, origin xyz=0.20 0 0.05 rpy=0 0 0
- added joint base_footprint_base_link_joint: type fixed, parent base_footprint, child base_link, origin xyz=0 0 0.1 rpy=0 0 0
- added joint base_laser_joint: type fixed, parent base_link, child laser, origin xyz=0 0 0.225 rpy=0 0 0
- added joint base_left_wheel_joint: type continuous, parent base_link, child left_wheel, origin xyz=-0.15 0.225 0 rpy=0 0 0, axis  0 1 0
- added joint base_right_wheel_joint: type continuous, parent base_link, child right_wheel, origin xyz=-0.15 -0.225 0 rpy=0 0 0, axis  0 1 0
